Commit message: add gunsight

File: pyflyt_dogfight/models/aggressor/aggressor.urdf (robot description, URDF)
Before this commit: robot aggressor, 8 links, 7 joints
Links:
- added link gunsight_link, mass 0; visual cylinder length=15.0 radius=0.3
Joints:
- added joint gunsight_joint: type fixed, parent base_link, child gunsight_link, origin xyz=7.5 0 0 rpy=0 1.571 0
